Commit message: Urdf using xacro and gazebo plugnin and camera used and learnt to code using gazebo tags and plugins

File: urdf_practice_Code/example_include.xacro (robot description, xacro)
@@ -1,38 +1,38 @@
-<?xml version = "1.0"?>
-<robot xmlns:xacro="http://www.ros.org/wiki/xacro">
-    <material name = "White">
+<?xml version="1.0"?>
+<robot xmlns:xacro="http://www.ros.org/wiki/xacro" >
+    <material name="white">
         <color rgba="1 1 1 1"/>
     </material>
-    <material name = "Orange">
+    <material name="orange">
         <color rgba="1 0.3 0.1 1"/>
     </material>
-    <material name = "Blue">
+    <material name="blue">
         <color rgba="0.2 0.2 1 1"/>
     </material>
-    <xacro:macro name="Inertial_Sphere" params = "mass radius *origin">
+    <xacro:macro name="inertial_sphere" params="mass radius *origin">
         <inertial>
-            <xacro:insert_block name = "origin"/>
-            <mass value = "${mass}"/>
-            <inertia ixx = "${(2/5) * mass * (radius * radius)}" ixy = "0.0" ixz = "0.0"
-                    iyy = "${(2/5) * mass * (radius * radius)}" iyz = "0.0"
-                    izz = "${(2/5) * mass * (radius * radius)}" />
+            <xacro:insert_block name="origin"/>
+            <mass value="${mass}" />
+            <inertia ixx="${(2/5) * mass * (radius*radius)}" ixy="0.0" ixz="0.0"
+                    iyy="${(2/5) * mass * (radius*radius)}" iyz="0.0"
+                    izz="${(2/5) * mass * (radius*radius)}" />
         </inertial>
     </xacro:macro>
-    <xacro:macro name="Inertial_Box" params = "mass x y z *origin">
+    <xacro:macro name="inertial_box" params="mass x y z *origin">
         <inertial>
-            <xacro:insert_block name = "origin"/>
-            <mass value = "${mass}"/>
-            <inertia ixx = "${(1/12) * mass * (y*y + z*z)}" ixy = "0.0" ixz = "0.0"
-                    iyy = "${(1/12) * mass * (x*x + z*z)}" iyz = "0.0"
-                    izz = "${(1/12) * mass * (x*x + y*y)}" />
+            <xacro:insert_block name="origin"/>
+            <mass value="${mass}" />
+            <inertia ixx="${(1/12) * mass * (y*y+z*z)}" ixy="0.0" ixz="0.0"
+                    iyy="${(1/12) * mass * (x*x+z*z)}" iyz="0.0"
+                    izz="${(1/12) * mass * (x*x+y*y)}" />
         </inertial>
     </xacro:macro>
-    <xacro:macro name="Inertial_Cylinder" params = "mass length radius *origin">
+    <xacro:macro name="inertial_cylinder" params="mass length radius *origin">
         <inertial>
-            <xacro:insert_block name = "origin"/>
-            <mass value = "${mass}"/>
-            <inertia ixx = "${(1/12) * mass * ((3 * radius * radius) + (length*length)) }" ixy = "0.0" ixz = "0.0"
-                    iyy = "${(1/12) * mass * ((3 * radius * radius) + (length*length)) }" iyz = "0.0"
-                    izz = "${(1/2) * mass * (radius * radius)}" />
+            <xacro:insert_block name="origin"/>
+            <mass value="${mass}" />
+            <inertia ixx="${(1/12) * mass * (3*radius*radius + length*length)}" ixy="0.0" ixz="0.0"
+                    iyy="${(1/12) * mass * (3*radius*radius + length*length)}" iyz="0.0"
+                    izz="${(1/2) * mass * (radius*radius)}" />
         </inertial>
     </xacro:macro>

File: urdf_practice_Code/example_robot.urdf.xacro (robot description, xacro)
@@ -1,6 +1,6 @@
 <?xml version="1.0"?>
-<robot xmlns:xacro="http://www.ros.org/wiki/xacro" name="robot">
-    <xacro:include filename="./example_include.xacro"/>
-    <link name="world"> </link>
+<robot xmlns:xacro="http://www.ros.org/wiki/xacro"  name="robot">
+    <xacro:include filename="example_include.xacro" />
+    <link name="world"></link>
     <joint name="base_joint" type="fixed">
         <origin xyz="1.5 1.0 0" rpy="0 0 0"/>
@@ -10,30 +10,30 @@
     <link name="base_link">
         <visual>
-            <origin xyz="0 0 0.5"" rpy="0 0 0"/>
+            <origin xyz="0 0 0.05" rpy="0 0 0"/>
             <geometry>
-                <box size="2.5 1.5 0.1"/>
+                <box size="2.5 1.5 0.1" />
             </geometry>
-            <material name="Green">
-                <color rgba="0.2 0.1 0.1 0.5"/>
+            <material name="green">
+                <color rgba="0.2 1 0.2 1"/>
             </material>
         </visual>
         <collision>
-            <origin xyz="0 0 0.5"" rpy="0 0 0"/>
+            <origin xyz="0 0 0.05" rpy="0 0 0"/>
             <geometry>
-                <box size="2.5 1.5 0.1"/>
+                <box size="2.5 1.5 0.1" />
             </geometry>
         </collision>
         <inertial>
-            <origin xyz="0 0 0.5"" rpy="0 0 0"/>
-            <mass value="12"/>
-            <inertia ixx="2.25" ixy="0.0" ixz="0.0" iyy="6.26" iyz="0.0" izz="8.5"/>
+            <origin xyz="0 0 0.05" rpy="0 0 0"/>
+            <mass value="12" />
+            <inertia ixx="2.26" ixy="0.0" ixz="0.0" iyy="6.26" iyz="0.0" izz="8.5" />
         </inertial>
     </link>
     <joint name="slider_joint" type="prismatic">
-        <origin xyz="1.25 0 0.1" rpy="0 0 0"/>
+        <origin xyz="-1.25 0 0.1" rpy="0 0 0"/>
         <parent link="base_link"/>
         <child link="slider_link"/>
         <axis xyz="1 0 0"/>
-        <limit lower="0" upper="2" velocity= "100" effort="200"/>
+        <limit lower="0" upper="2" velocity="100" effort="100"/>
     </joint>
     <link name="slider_link">
@@ -41,47 +41,47 @@
             <origin xyz="0 0 0.075" rpy="0 0 0"/>
             <geometry>
-                <box size="0.5 0.25 0.15"/>
+                <box size="0.5 0.25 0.15" />
             </geometry>
-            <material name="Blue"/>
+            <material name="blue" />
         </visual>
         <collision>
             <origin xyz="0 0 0.075" rpy="0 0 0"/>
             <geometry>
-                <box size="0.5 0.25 0.15"/>
+                <box size="0.5 0.25 0.15" />
             </geometry>
         </collision>
-        <xacro:Inertial_Box mass="0.5" x="0.5" y="0.25" z="0.15">
+        <xacro:inertial_box mass="0.5" x="0.5" y="0.25" z="0.15">
             <origin xyz="0 0 0.075" rpy="0 0 0"/>
-        </xacro:Inertial_Box>
+        </xacro:inertial_box>
     </link>
-   <joint name="arm_joint" type="revolute">
-        <origin xyz="0.25 0.0 0.15" rpy="0 0 0"/>
+    <joint name="arm_joint" type="revolute">
+        <origin xyz="0.25 0 0.15" rpy="0 0 0"/>
         <parent link="slider_link"/>
         <child link="arm_link"/>
         <axis xyz="0 -1 0"/>
-        <limit lower="0" upper="${pi / 2}" velocity="100" effort="100"/>
+        <limit lower="0" upper="${pi/2}" velocity="100" effort="100"/>
     </joint>
-    <xacro:property name="arm_length" value="1"/>
-    <xacro:property name="arm_radius" value="0.1"/>
+    <xacro:property name="arm_length" value="1" />
+    <xacro:property name="arm_radius" value="0.1" />
     <link name="arm_link">
         <visual>
-            <origin xyz="${arm_length / 2} 0 0" rpy="0 ${pi/2} 0"/>
+            <origin xyz="${arm_length/2} 0 0" rpy="0 ${pi/2} 0"/>
             <geometry>
-                <cylinder length="${arm_length}" radius="${arm_radius}"/>
+                <cylinder length="${arm_length}" radius="${arm_radius}" />
             </geometry>
-            <material name="Orange"/>
+            <material name="orange" />
         </visual>
         <collision>
-            <origin xyz="${arm_length / 2} 0 0" rpy="0 ${pi/2} 0"/>
+            <origin xyz="${arm_length/2} 0 0" rpy="0 ${pi/2} 0"/>
             <geometry>
-                <cylinder length="${arm_length}" radius="${arm_radius}"/>
+                <cylinder length="${arm_length}" radius="${arm_radius}" />
             </geometry>
         </collision>
-        <xacro:Inertial_Cylinder mass="1.0" length="${arm_length}" radius="${arm_radius}">
-            <origin xyz="${arm_length / 2} 0 0" rpy="0 ${pi/2} 0"/>
-        </xacro:Inertial_Cylinder>
+        <xacro:inertial_cylinder mass="1.0" length="${arm_length}" radius="${arm_radius}">
+            <origin xyz="${arm_length/2} 0 0" rpy="0 ${pi/2} 0"/>
+        </xacro:inertial_cylinder>
     </link>
     <joint name="camera_joint" type="fixed">
-        <origin xyz="${arm_length} 0 ${arm_radius + 0.75}" rpy="0 0 0"/>
+        <origin xyz="${arm_length} 0 ${arm_radius + 0.075}" rpy="0 0 0"/>
         <parent link="arm_link"/>
         <child link="camera_link"/>
@@ -89,19 +89,26 @@
     <link name="camera_link">
         <visual>
-            <origin xyz="0.03 0 0" rpy="0 0 0"/>
+            <origin xyz="-0.03 0 0" rpy="0 0 0"/>
             <geometry>
-                <box size=" 0.06 0.15 0.15"/>
+                <box size="0.06 0.15 0.15" />
             </geometry>
-            <material name="White"/>
+            <material name="white" />
+        </visual>
+        <visual>
+            <origin xyz="0.03 0 0" rpy="0 ${pi/2} 0"/>
+            <geometry>
+                <cylinder length="0.06" radius="0.04" />
+            </geometry>
+            <material name="blue" />
         </visual>
         <collision>
-            <origin xyz="0.03 0 0" rpy="0 0 0"/>
+            <origin xyz="0.0 0 0" rpy="0 0 0"/>
             <geometry>
-                <box size=" 0.06 0.15 0.15"/>
+                <box size="0.12 0.15 0.15" />
             </geometry>
         </collision>
-        <xacro:Inertial_Box mass="0.1" x="0.12" y="0.15" z="0.15">
-            <origin xyz="0.03 0 0" rpy="0 0 0"/>
-        </xacro:Inertial_Box>
+        <xacro:inertial_box mass="0.1" x="0.12" y="0.15" z="0.15">
+            <origin xyz="0.0 0 0" rpy="0 0 0"/>
+        </xacro:inertial_box>
     </link>
 </robot>
